File: kicad-project/garage-door-controller.kicad_pcb (KiCad board)
At the start: 2 copper layers, 100 x 100 mm, 144 parts, among them CN1 PSU, CN2 Motor, CN3 Tacho, CN4 RF-RX480E, CN5 RF-HCS301, CN9 UART, Q1 AO3400A, Q10 SL142N06Q, Q11 SL142N06Q, Q12 SL142N06Q, Q2 SS8050, Q3 IRFZ44NPBF, Q4 SL142N06Q, Q5 SS8050, Q6 SS8550, Q7 SS8050, Q8 SS8050, Q9 SL142N06Q, SW1 TS-1187A-B-A-B, SW2 TS-1187A-B-A-B, U1 EL3H7(B)(TA)-G, U10 SN74HCS08DR, U2 EL3H7(B)(TA)-G, U3 EL3H7(B)(TA)-G, U4 EL3H7(B)(TA)-G, U5 EL3H7(B)(TA)-G, U6 XL1509-5.0E1, U7 AMS1117-3.3, U8 ESP32-WROOM-32E(4MB), U9 DRV8701PRGET, X1 WJ500V-5.08-3P-14-00A, X2 WJ500V-5.08-3P-14-00A, X3 WJ500V-5.08-2P-14-00A, X4 WJ500V-5.08-3P-14-00A

Commit message: minor
Parts:
- added R56: 10k, easyeda2kicad:R0603, F.Cu at (134.0, 113.5)
- moved R37 35.9 mm to (134.4, 98.7), turned to 180 degrees
- moved R36 35.9 mm to (134.4, 95.2), turned to 180 degrees
- moved R35 35.9 mm to (134.4, 91.6), turned to 180 degrees
- moved JP1 25.7 mm to (130.2, 88.0), turned to 180 degrees
- moved JP2 25.7 mm to (130.2, 91.6), turned to 180 degrees
- moved JP3 25.7 mm to (130.2, 95.2), turned to 180 degrees
- moved JP4 25.7 mm to (130.2, 98.7), turned to 180 degrees
- moved JP5 25.7 mm to (130.2, 102.2), turned to 180 degrees
- moved C24 2.05 mm to (132.0, 115.8), turned to -90 degrees
Connections:
- net Net-(Q3-G) renamed /L_GATE_DRV
- U10 pad 10: +3V3 -> Net-(U10-3A)
- U10 pad 12: +3V3 -> Net-(U10-3A)
- U10 pad 8: +3V3 -> Net-(U10-3A)
- U10 pad 9: +3V3 -> Net-(U10-3A)
Routing:
- net +3V3: track 228.8 -> 214.4 mm
- net Net-(U10-3A): track 0.00 -> 13.9 mm
- net /AVDD: track 37.7 -> 48.2 mm, vias 0 -> 2
- net /IDRIVE: track 34.0 -> 24.0 mm
- net /IDRV2: track 5.66 -> 2.75 mm
- net /IDRV3: track 5.47 -> 2.75 mm
- net /IDRV4: track 5.26 -> 2.75 mm
- net GND: vias 563 -> 73
Other:
- board text added: "Flash"
- board text added: "Reset"

Commit message: upd
Routing:
- net +3V3: track 214.4 -> 216.2 mm, vias 5 -> 4
- net /AVDD: track 48.2 -> 47.1 mm

Commit message: upd
Parts:
- moved CN3 15.8 mm to (99.0, 91.7), turned to 0 degrees
- moved R38 9.12 mm to (102.2, 95.5), turned to -90 degrees
- moved RV1 4.91 mm to (105.0, 103.0), turned to -90 degrees
- moved R52 1.65 mm to (127.8, 134.2), turned to 10 degrees
- moved R55 1.27 mm to (124.9, 126.5), turned to 35 degrees
- moved R51 1.15 mm to (127.2, 132.2), turned to 15 degrees
- moved R26 0.79 mm to (79.2, 109.0), turned to -135 degrees
- moved R53 0.65 mm to (126.8, 130.2), turned to 20 degrees
- moved JP8 0.50 mm to (119.5, 106.2)
- moved R27 0.35 mm to (78.8, 114.0), turned to -135 degrees
- moved R54 0.10 mm to (126.0, 128.2), turned to 25 degrees
Routing:
- net MOTOR_TACHO: track 36.8 -> 46.8 mm
- net +5V: track 33.0 -> 24.3 mm
- net +3V3: track 216.2 -> 210.8 mm
- net /AVDD: track 47.1 -> 43.8 mm
- net /RF_D0: track 19.7 -> 16.7 mm
- net /RF_D1: track 19.9 -> 17.3 mm
- net /MCU_PSU_ON: track 79.9 -> 77.6 mm
- net /RF_D2: track 20.1 -> 18.0 mm
- net +24V: track 145.1 -> 147.1 mm
- net REQ_TOGGLE: track 37.4 -> 35.4 mm
- net /RF_VT_MCU: track 10.2 -> 8.42 mm
- net LIM_TOP: track 84.6 -> 86.4 mm
- net /RF_D0_MCU: track 8.91 -> 10.5 mm
- net /L_V_FLW: track 7.25 -> 8.80 mm
- net /VREF_VAR: track 10.2 -> 8.71 mm
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- added copper zone on F.Cu, net LIM_TOP
Other:
- board text added: "GND"
- board text added: "GND +24 +36 ENA_36"
- board text added: "RX"
- board text added: "TX"
- board text removed: "+VM"
- board text removed: "Boot Flash"
- board text removed: "EN_36 +36 +24 GND"
- board text removed: "GND PWM +RLY BTM +V TOP DWN +V UP +V BTN"
- board text removed: "GND RX TX 3.3"
- board text removed: "T"

Commit message: upd
Parts:
- R13: value 2.2k -> 2k2
- moved R24 1.68 mm to (79.0, 98.5), turned to 90 degrees
- moved R25 1.68 mm to (79.0, 103.5), turned to 90 degrees
Routing:
- net LIM_TOP: track 86.4 -> 84.5 mm
- net LIM_BOTTOM: track 80.0 -> 78.1 mm
- net GND: vias 83 -> 414
Other:
- board text added: "Garage door controller 2.0 - DRV8701 motor driver 36V/7A - convenient light - limit switches github.com/latonita"
- board text added: "PWR"
- board text added: "fix"
- board text added: "var"
- board text removed: "Garage door controller - DRV8701 motor driver 36V/7A max - convenient light - limit switches github.com/latonita"
