File: kicad-project/garage-door-controller.kicad_pcb (KiCad board)
At the start: 2 copper layers, 100 x 100 mm, 147 parts, among them CN1 PSU, CN2 UART, CN3 Tacho, CN4 Motor, CN5 RF-RX480E, CN6 RF-HCS301, Q1 AO3400A, Q10 SL142N06Q, Q11 SL142N06Q, Q12 SL142N06Q, Q2 SS8050, Q3 IRFZ44NPBF, Q4 SL142N06Q, Q5 SS8050, Q6 SS8550, Q7 SS8050, Q8 SS8050, Q9 SL142N06Q, SW1 TS-1187A-B-A-B, SW2 TS-1187A-B-A-B, U1 EL3H7(B)(TA)-G, U10 SN74HCS08DR, U2 EL3H7(B)(TA)-G, U3 EL3H7(B)(TA)-G, U4 EL3H7(B)(TA)-G, U5 EL3H7(B)(TA)-G, U6 XL1509-5.0E1, U7 AMS1117-3.3, U8 ESP32-WROOM-32E(4MB), U9 DRV8701PRGET, X1 WJ500V-5.08-3P-14-00A, X2 WJ500V-5.08-3P-14-00A, X3 WJ500V-5.08-2P-14-00A, X4 WJ500V-5.08-3P-14-00A

Commit message: upd
Parts:
- removed TP2, TP3: TestPoint, easyeda2kicad:TestPoint_Pad_D1.5mm
- moved R36 26.6 mm to (122.5, 96.8), turned to 0 degrees
- moved SW1 3.95 mm to (103.4, 112.9), turned to -90 degrees
- moved C10 1.05 mm to (97.7, 120.4)
- moved R33 1.05 mm to (97.7, 115.9)
- moved R34 1.05 mm to (97.7, 118.1)
Connections:
- net /IDRV2 renamed Net-(JP5-A)
- net /IDRV3 renamed Net-(JP6-A)
- net /IDRV4 renamed Net-(JP7-A)
- net /SN_MOTOR_TACHO renamed /AND_TACHO
- net /SN_PWM_DOWN renamed /AND_PWM_DOWN
- net /SN_PWM_UP renamed /AND_PWM_UP
- net LIM_BOTTOM renamed IN_LIM_BOTTOM
- net LIM_TOP renamed IN_LIM_TOP
- net MOTOR_TACHO renamed /TACHO
- net REQ_DOWN renamed IN_DOWN
- net REQ_TOGGLE renamed IN_TOGGLE
- net REQ_UP renamed IN_UP
- D1 pad 2: LIGHT_LOW -> LIGHT_SINK
- Q4 pad 5: LIGHT_LOW -> LIGHT_SINK
- Q4 pad 6: LIGHT_LOW -> LIGHT_SINK
- Q4 pad 7: LIGHT_LOW -> LIGHT_SINK
- Q4 pad 8: LIGHT_LOW -> LIGHT_SINK
- Q4 pad 9: LIGHT_LOW -> LIGHT_SINK
- R36 pad 1: +3V3 -> /DVDD
- X4 pad 2: LIGHT_LOW -> LIGHT_SINK
Routing:
- net +3V3: track 225.3 -> 211.8 mm
- net /DVDD: track 11.2 -> 17.2 mm, vias 0 -> 2
- net Net-(SW1-C): track 8.69 -> 12.5 mm, vias 0 -> 2
- net +36V: track 3.20 -> 5.63 mm
- net /MCU_PWM_UP: track 28.8 -> 26.8 mm
- net /MCU_PWM_DN: track 23.8 -> 21.8 mm
- net /BOOT_MODE: track 8.98 -> 10.0 mm
- net GND: vias 96 -> 100
- added copper zone on F.Cu, net LIGHT_SINK
- removed copper zone on F.Cu, net LIGHT_LOW
