File: kicad-project/garage-door-controller.kicad_sch (KiCad schematic)
At the start: 145 parts, among them CN1 PSU, CN2 Motor, CN3 Tacho, CN4 RF-RX480E, CN5 RF-HCS301, CN9 UART, Q1 AO3400A, Q10 SL142N06Q, Q11 SL142N06Q, Q12 SL142N06Q, Q2 SS8050, Q3 IRFZ44NPBF, Q4 SL142N06Q, Q5 SS8050, Q6 SS8550, Q7 SS8050, Q8 SS8050, Q9 SL142N06Q, SW1 TS-1187A-B-A-B, SW2 TS-1187A-B-A-B, U1 EL3H7(B)(TA)-G, U10 SN74HCS08DR, U2 EL3H7(B)(TA)-G, U3 EL3H7(B)(TA)-G, U4 EL3H7(B)(TA)-G, U5 EL3H7(B)(TA)-G, U6 XL1509-5.0E1, U7 AMS1117-3.3, U8 ESP32-WROOM-32E(4MB), U9 DRV8701PRGET, X1 WJ500V-5.08-3P-14-00A, X2 WJ500V-5.08-3P-14-00A, X3 WJ500V-5.08-2P-14-00A, X4 WJ500V-5.08-3P-14-00A

Commit message: minor
Parts:
- added R56: 10k, easyeda2kicad:R0603, symbol easyeda2kicad:0603WAF1002T5E
- SW1: Label (none) -> Flash
- SW2: Label (none) -> Reset
Connections:
- net +3V3: now also R56.2; no longer U10.10 (3B), U10.12 (4A), U10.8 (3Y), U10.9 (3A)
- net L_GATE_DRV: now also Q3.1 (G), Q4.4 (G), R20.1
- new net: R56.1, U10.10 (3B), U10.12 (4A), U10.8 (3Y), U10.9 (3A)
Other:
- moved on the sheet: C5, C8

Commit message: upd
Other:
- note added: "Convenient light PWM or External relay control"
- note added: "Motor H-bridge"
Changed lines of the file:
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@@
 		)
 	)
+	(text "Motor H-bridge"
+		(exclude_from_sim no)
+		(at 300.99 131.318 0)
+		(effects
+			(font
+				(size 2 2)
+				(thickness 0.6)
+				(bold yes)
+			)
+			(justify left top)
+		)
+	)
 	(text "Top/Bottom"
 		(exclude_from_sim no)
@@
 		)
 	)
+	(text "Convenient light PWM or External relay control"
+		(exclude_from_sim no)
+		(at 168.91 211.074 0)
+		(effects
+			(font
+				(size 2 2)
+				(thickness 0.4)
+				(bold yes)
+			)
+			(justify left)
+		)
+	)
 	(text "+24 and LIGHT_LOW are \nfor external 24V relay\n\nLIGHT_LOW and GND can \nbe used for PWM ground, \nexternal supply needed."
 		(exclude_from_sim no)
@@
 		)
 	)
-	(text_box "Convenient light PWM or External relay control"
-		(exclude_from_sim no)
-		(at 167.64 208.28 0)
-		(size 129.54 71.12)
-		(margins 0.9525 0.9525 0.9525 0.9525)
-		(stroke
-			(width 0)
-			(type solid)
-		)
-		(fill
-			(type none)
-		)
-		(effects
-			(font
-				(size 1.27 1.27)
-			)
-			(justify left top)
-		)
-	)
 	(text_box "DC-DC\n5V0\n3V3"
 		(exclude_from_sim no)
@@
 		)
 	)
-	(text_box "Motor H-bridge"
-		(exclude_from_sim no)
-		(at 297.18 128.27 0)
-		(size 107.95 76.708)
-		(margins 0.9525 0.9525 0.9525 0.9525)
-		(stroke
-			(width 0)
-			(type solid)
-		)
-		(fill
-			(type none)
-		)
-		(effects
-			(font
-				(size 1.27 1.27)
-			)
-			(justify left top)
-		)
-	)
 	(text_box "Extrn PSU\n24V\n36V off/on"
 		(exclude_from_sim no)
@@
 		)
 	)
+	(polyline
+		(pts
+			(xy 299.72 128.27) (xy 299.72 204.47)
+		)
+		(stroke
+			(width 0)
+			(type default)
+		)
+	)
 	(wire
 		(pts
@@
 		)
 	)
+	(polyline
+		(pts
+			(xy 297.18 279.4) (xy 297.18 208.28)
+		)
+		(stroke
+			(width 0)
+			(type default)
+		)
+	)
 	(wire
 		(pts
@@
 		)
 	)
+	(polyline
+		(pts
+			(xy 167.64 279.4) (xy 297.18 279.4)
+		)
+		(stroke
+			(width 0)
+			(type default)
+		)
+	)
 	(wire
 		(pts
@@
 		)
 	)
+	(polyline
+		(pts
+			(xy 405.13 204.47) (xy 299.72 204.47)
+		)
+		(stroke
+			(width 0)
+			(type default)
+		)
+	)
 	(wire
 		(pts
@@
 		)
 	)
+	(polyline
+		(pts
+			(xy 405.13 128.27) (xy 405.13 204.47)
+		)
+		(stroke
+			(width 0)
+			(type default)
+		)
+	)
 	(wire
 		(pts
@@
 		)
 	)
+	(polyline
+		(pts
+			(xy 299.72 128.27) (xy 405.13 128.27)
+		)
+		(stroke
+			(width 0)
+			(type default)
+		)
+	)
 	(wire
 		(pts
@@
 	(polyline
 		(pts
+			(xy 167.64 208.28) (xy 297.18 208.28)
+		)
+		(stroke
+			(width 0)
+			(type default)
+		)
+	)
+	(polyline
+		(pts
 			(xy 212.725 151.765) (xy 212.09 151.13)
 		)
@@
 		)
 	)
+	(polyline
+		(pts
+			(xy 167.64 208.28) (xy 167.64 279.4)
+		)
+		(stroke
+			(width 0)
+			(type default)
+		)
+	)
 	(wire
 		(pts
@@
 					(size 1.27 1.27)
 				)
+				(hide yes)
 			)
 		)
@@
 					(size 1.27 1.27)
 				)
+				(hide yes)
 			)
 		)

Commit message: upd
Parts:
- R13: value 2.2k -> 2k2
Changed lines of the file:
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@@
 			)
 		)
-		(property "Description" ""
+		(property "Description" "100mW Thick Film Resistors 75V ±100ppm/℃ ±1% 2.2kΩ 0603 Chip Resistor - Surface Mount ROHS"
 			(at 113.03 205.74 0)
 			(effects
@@
 			)
 		)
-		(property "Description" ""
+		(property "Description" "100mW Thick Film Resistors 75V ±100ppm/℃ ±1% 2.2kΩ 0603 Chip Resistor - Surface Mount ROHS"
 			(at 43.18 266.7 0)
 			(effects
@@
 			)
 		)
-		(property "Description" ""
+		(property "Description" "100mW Thick Film Resistors 75V ±100ppm/℃ ±1% 2.2kΩ 0603 Chip Resistor - Surface Mount ROHS"
 			(at 43.18 233.68 0)
 			(effects
@@
 			)
 		)
-		(property "Description" ""
+		(property "Description" "100mW Thick Film Resistors 75V ±100ppm/℃ ±1% 2.2kΩ 0603 Chip Resistor - Surface Mount ROHS"
 			(at 43.18 254 0)
 			(effects
@@
 			)
 		)
-		(property "Description" ""
+		(property "Description" "100mW Thick Film Resistors 75V ±100ppm/℃ ±1% 2.2kΩ 0603 Chip Resistor - Surface Mount ROHS"
 			(at 43.18 220.98 0)
 			(effects
@@
 			)
 		)
-		(property "Description" ""
+		(property "Description" "100mW Thick Film Resistors 75V ±100ppm/℃ ±1% 2.2kΩ 0603 Chip Resistor - Surface Mount ROHS"
 			(at 113.03 228.6 0)
 			(effects
@@
 			)
 		)
-		(property "Value" "2.2k"
+		(property "Value" "2k2"
 			(at 181.61 234.95 0)
 			(effects
@@
 			)
 		)
-		(property "Description" ""
+		(property "Description" "100mW Thick Film Resistors 75V ±100ppm/℃ ±1% 2.2kΩ 0603 Chip Resistor - Surface Mount ROHS"
 			(at 113.03 241.3 0)
 			(effects
@@
 			)
 		)
-		(property "Description" ""
+		(property "Description" "100mW Thick Film Resistors 75V ±100ppm/℃ ±1% 2.2kΩ 0603 Chip Resistor - Surface Mount ROHS"
 			(at 113.03 193.04 0)
 			(effects
@@
 			)
 		)
-		(property "Description" ""
+		(property "Description" "100mW Thick Film Resistors 75V ±100ppm/℃ ±1% 2.2kΩ 0603 Chip Resistor - Surface Mount ROHS"
 			(at 43.18 190.5 0)
 			(effects
@@
 			)
 		)
-		(property "Description" ""
+		(property "Description" "100mW Thick Film Resistors 75V ±100ppm/℃ ±1% 2.2kΩ 0603 Chip Resistor - Surface Mount ROHS"
 			(at 43.18 203.2 0)
 			(effects
