File: kicad-project/garage-door-controller.kicad_sch (KiCad schematic)
At the start: 148 parts, among them CN1 PSU, CN2 UART, CN3 Tacho, CN4 Motor, CN5 RF-RX480E, CN6 RF-HCS301, Q1 AO3400A, Q10 SL142N06Q, Q11 SL142N06Q, Q12 SL142N06Q, Q2 SS8050, Q3 IRFZ44NPBF, Q4 SL142N06Q, Q5 SS8050, Q6 SS8550, Q7 SS8050, Q8 SS8050, Q9 SL142N06Q, SW1 TS-1187A-B-A-B, SW2 TS-1187A-B-A-B, U1 EL3H7(B)(TA)-G, U10 SN74HCS08DR, U2 EL3H7(B)(TA)-G, U3 EL3H7(B)(TA)-G, U4 EL3H7(B)(TA)-G, U5 EL3H7(B)(TA)-G, U6 XL1509-5.0E1, U7 AMS1117-3.3, U8 ESP32-WROOM-32E(4MB), U9 DRV8701PRGET, X1 WJ500V-5.08-3P-14-00A, X2 WJ500V-5.08-3P-14-00A, X3 WJ500V-5.08-2P-14-00A, X4 WJ500V-5.08-3P-14-00A

Commit message: upd
Parts:
- removed TP2, TP3: TestPoint, easyeda2kicad:TestPoint_Pad_D1.5mm, symbol easyeda2kicad:TestPoint
- CN2: symbol Connector:Conn_01x04_Pin -> Connector_Generic:Conn_01x04; now in the parts list
Connections:
- net +3V3: no longer R36.1
- net DVDD: now also R36.1
- net GND: no longer H1.1, H2.1, H3.1, H4.1
- net IDRV2: no longer names the net of JP5.1 (A), R53.2
- net IDRV3: no longer names the net of JP6.1 (A), R54.2
- net IDRV4: no longer names the net of JP7.1 (A), R55.2
- net LIGHT_LOW renamed LIGHT_SINK
- net LIM_BOTTOM renamed IN_LIM_BOTTOM
- net LIM_TOP renamed IN_LIM_TOP
- net MOTOR_TACHO renamed TACHO
- net REQ_DOWN renamed IN_DOWN
- net REQ_TOGGLE renamed IN_TOGGLE
- net REQ_UP renamed IN_UP
- net SN_MOTOR_TACHO renamed AND_TACHO
- net SN_PWM_DOWN renamed AND_PWM_DOWN
- net SN_PWM_UP renamed AND_PWM_UP
- no-connect marks 14 -> 17
Other:
- note added: "All optocouplers are EL3H7(B)(TA)-G"
- note added: "I max = 7A P rsens = I x I x R = 7 x 7 x 0.010R = 0.5W U rsens = I x R = 7 x 0.010 = 0.07V SO = Av * U shunt = 20 x 0.07V = 1.4V"
- note added: "Mosfets - SL142N06Q Diodes - SS36 Bulk caps are 50V"
- note added: "Motor"
- note added: "Other MOSFET options: --------------------- NVMFS6H824NT1G 80V, 4.5mR, 38nC $1.53 CSD18531Q5A 60V, 3.5mR, 36nc $1.13 SL142N06Q 60V 2.6mR 45nC $0.47 SP60N02BGNK 60V 2.3mR 53nC $0.49"
- note added: "PSU control"
- note added: "UART header"
- note added: "hall sensor requirement"
- note added: "optionally go to MCU ADC"
- note added: "to MCU"
- note removed: "MOSFET options: NVMFS6H824NT1G 80V, 4.5mR, 38nC $1.53 CSD18531Q5A 60V, 3.5mR, 36nc $1.13 SL142N06Q 60V 2.6mR 45nC $0.47 SP60N02BGNK 60V 2.3mR 53nC $0.49"
- note removed: "Motor PSU control"
- note removed: "P r_sens = I^2 x R = 49 * 0.010 = 0.5W"
- note removed: "SO = Av * U shunt = 20 x 0.07 V = 1.4 V"
- note removed: "U shunt = I * R = 7 * 0.010 = 0.07 V"
- note removed: "Unused pins to VCC"
- note removed: "optional to MCU ADC"
- moved on the sheet: C1, C10, C11, C12, C13, C14, C15, C16, C17, C18, C19, C2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
